File: PCBs/Conductivity_Sensor/Conductivity_Sensor_V1/Conductivity_Sensor_V1_with_transistor/Conductivity_Sensor_V1.kicad_pcb (KiCad board)
At the start: 2 copper layers, 80.3 x 105.5 mm, 26 parts, among them J10 Optical density connector, J11 Conn_02x02_Top_Bottom, J12 Conn_02x04_Counter_Clockwise, J13 Solder lead 2, J14 Solder lead 1, J2 Test pad 5v+, J3 Test pad GND, J4 Test pad 12v+, J5 Test pad GND, J6 Screen connector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

Commit message: up
Parts:
- moved J2 58.4 mm to (-43.2, 179.1)
- moved J4 49.0 mm to (-21.6, 185.4)
- moved J14 31.1 mm to (-8.89, 233.7)
- moved J13 28.3 mm to (-10.2, 185.4)
- moved J3 14.0 mm to (-42.8, 185.6)
- moved J5 14.0 mm to (-31.6, 185.6)
Connections:
- C3 pad 1: OUT1 -> Net-(C3-Pad1)
- J10 pad 5: (no net) -> Net-(J10-Pad5)
- J10 pad 6: (no net) -> Net-(J10-Pad6)
- J11 pad 1: OUT1 -> Net-(C3-Pad1)
- J11 pad 2: OUT1 -> Net-(C3-Pad1)
- J11 pad 3: OUT1 -> Net-(J11-Pad3)
- J12 pad 8: (no net) -> Net-(J12-Pad8)
- Q1 pad 3: OUT1 -> Net-(J11-Pad3)
- U2 pad 10: (no net) -> Net-(U2-Pad10)
- U2 pad 12: (no net) -> Net-(U2-Pad12)
- U2 pad 13: (no net) -> Net-(U2-Pad13)
- U2 pad 16: (no net) -> Net-(U2-Pad16)
- U2 pad 17: (no net) -> Net-(U2-Pad17)
- U2 pad 18: (no net) -> Net-(U2-Pad18)
- U2 pad 19: (no net) -> Net-(U2-Pad19)
- U2 pad 2: (no net) -> Net-(U2-Pad2)
- U2 pad 24: (no net) -> Net-(U2-Pad24)
- U2 pad 25: (no net) -> Net-(U2-Pad25)
- U2 pad 3: (no net) -> Net-(U2-Pad3)
- U2 pad 30: (no net) -> Net-(U2-Pad30)
- U2 pad 6: (no net) -> Net-(U2-Pad6)
- U2 pad 7: (no net) -> Net-(U2-Pad7)
- U2 pad 8: (no net) -> Net-(U2-Pad8)
- U2 pad 9: (no net) -> Net-(U2-Pad9)
- U3 pad 2: OUT1 -> Net-(C3-Pad1)
- U3 pad 6: OUT1 -> Net-(C3-Pad1)
Other:
- board text added: "0.1µF"
- board text added: "1.5K"
- board text added: "1M ohm"
- board text added: "1k Ohm"
- board text added: "1µf"
- board text added: "510"
- board text added: "EC Meter + OD V1.0 IGEM Bettancourt 2022"
- board text added: "GND"
- board text added: "R Divider"
- board text added: "Regulated 5V +"
- board text added: "Sensor Lead 1"
- board text added: "Sensor Lead 2"
- board text added: "Test Pads"
- board text added: "Transistor"
- board text added: "v+ 12V"

Commit message: up
Parts:
- moved J2 4.61 mm to (-38.6, 178.9)
- moved U2 0.96 mm to (11.5, 211.9)
Routing:
- net GND: track 0.00 -> 185.1 mm
- net OUT1: track 0.00 -> 151.7 mm, vias 0 -> 1
- net OUT2: track 0.00 -> 140.4 mm
- net REGULATED_5V+: track 0.00 -> 111.6 mm
- net LED4: track 0.00 -> 99.9 mm
- net LED2: track 0.00 -> 92.3 mm, vias 0 -> 1
- net LED3: track 0.00 -> 90.2 mm
- net LED1: track 0.00 -> 84.3 mm
- net V+_12V: track 0.00 -> 80.7 mm
- net ESP8266_3V: track 0.00 -> 72.6 mm
- net 555_out: track 0.00 -> 70.3 mm
- net Transistor_Control: track 0.00 -> 62.5 mm
- net LED6: track 0.00 -> 57.1 mm
- net A0: track 0.00 -> 55.1 mm
- net SCL: track 0.00 -> 54.1 mm
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Other:
- outline, holes or cut-outs redrawn
