File: PCBs/Conductivity_Sensor/Conductivity_Sensor_V1/Conductivity_Sensor_V1_LED_BOARD/LED_BOARD_V1.kicad_pcb (KiCad board)
At the start: 2 copper layers, 95.5 x 80.3 mm, 13 parts, among them J1 Conn_02x04_Counter_Clockwise

Commit message: up
Routing:
- net GND: track 0.00 -> 138.6 mm
- net LED6: track 0.00 -> 66.1 mm
- net LED1: track 0.00 -> 65.1 mm
- net LED2: track 0.00 -> 63.7 mm
- net LED4: track 0.00 -> 62.6 mm
- net LED3: track 0.00 -> 56.8 mm
- net LED5: track 0.00 -> 56.8 mm, vias 0 -> 1
- net Net-(D6-Pad1): track 0.00 -> 30.8 mm
- net Net-(D3-Pad1): track 0.00 -> 28.0 mm
- net Net-(D5-Pad1): track 0.00 -> 20.7 mm
- net Net-(D4-Pad1): track 0.00 -> 15.5 mm
- net Net-(D1-Pad1): track 0.00 -> 12.8 mm
- net Net-(D2-Pad1): track 0.00 -> 9.53 mm
